File: Detector/Detector.kicad_pcb (KiCad board)
At the start: 2 copper layers, 100 x 100 mm, 52 parts, among them J1 Power, J2 Signal, Q1 2N3904, Q2 2N3904, Q3 2N3904, Q4 2N3904, Q5 2N3906, Q6 2N3906, Q7 2N3906, Q8 2N3904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

Commit message: More placement and routing
Parts:
- D10: value LED C1 -> C-1
- D11: value LED D2 -> D-2
- D12: value LED D1 -> D-1
- D5: value LED A2 -> A-2
- D6: value LED A1 -> A-1
- D7: value LED B2 -> B-2
- D8: value LED B1 -> B-1
- D9: value LED C2 -> C-2
- moved R17 132.2 mm to (135.0, 119.8), turned to 90 degrees
- moved R4 125.6 mm to (94.0, 94.6), turned to 90 degrees
- moved R22 118.8 mm to (108.0, 119.2), turned to -90 degrees
- moved R23 110.8 mm to (98.0, 119.2), turned to -90 degrees
- moved J1 103.2 mm to (156.5, 128.6), turned to -90 degrees
- moved R21 60.9 mm to (94.0, 65.5), turned to 90 degrees
- moved J2 40.0 mm to (141.9, 128.6), turned to -90 degrees
- moved R3 38.8 mm to (103.0, 126.8), turned to 90 degrees
- moved R14 38.8 mm to (182.0, 98.0), turned to -90 degrees
- moved R15 36.4 mm to (99.0, 105.6), turned to 90 degrees
- moved R1 34.4 mm to (187.0, 94.6)
- moved R10 34.2 mm to (177.0, 98.0), turned to -90 degrees
- moved R2 29.2 mm to (177.0, 125.8), turned to 90 degrees
- moved Q2 28.6 mm to (178.0, 112.0)
- moved R11 27.8 mm to (104.0, 105.6), turned to 90 degrees
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Routing:
- net Net-(Q9-C): track 0.00 -> 77.0 mm
- net /LED4: track 0.00 -> 62.4 mm
- net Net-(D11-A): track 0.00 -> 44.0 mm
- net /LED3: track 0.00 -> 30.5 mm
- net /DET2: track 0.00 -> 26.8 mm
- net Net-(D1-A): track 48.7 -> 27.6 mm
- net /DET1: track 0.00 -> 19.4 mm
- net Net-(D10-A): track 19.0 -> 0.00 mm
- net Net-(D1-K): track 17.8 -> 0.00 mm
- net Net-(Q1-C): track 16.5 -> 0.00 mm
- net Net-(Q3-C): track 0.00 -> 14.5 mm
- net Net-(Q8-B): track 13.7 -> 0.00 mm
- net /38KHz: track 0.00 -> 11.7 mm
- net Net-(D10-K): track 0.00 -> 11.5 mm
- net Net-(Q8-C): track 11.4 -> 0.00 mm
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Other:
- outline, holes or cut-outs redrawn
- board text added: "38KHz"
- board text added: "DET 1"
- board text added: "DET 2"
- board text added: "LED A"
- board text added: "LED B"
- board text added: "LED C"
- board text added: "LED D"

Commit message: Update detector borad
Parts:
- D10: value C-1 -> LED C1
- D11: value D-2 -> LED D2
- D12: value D-1 -> LED D1
- D3: footprint LED_THT:LED_D5.0mm_Horizontal_O3.81mm_Z9.0mm -> LED_THT:LED_D5.0mm_Horizontal_O3.81mm_Z3.0mm
- D5: value A-2 -> LED A2
- D6: value A-1 -> LED A1
- D7: value B-2 -> LED B2
- D8: value B-1 -> LED B1
- D9: value C-2 -> LED C2
- U1, U2: value TSOP343xx -> TSOP34338
- moved R22 42.9 mm to (150.8, 116.0), turned to 0 degrees
- moved R9 5.16 mm to (177.0, 87.0)
- moved R13 4.92 mm to (172.0, 87.0)
- moved R17 3.81 mm to (135.0, 116.0), turned to 180 degrees
- moved Q5 3.08 mm to (142.1, 116.0)
- moved Q2 2.67 mm to (175.3, 112.0), turned to 0 degrees
- moved Q3 2.60 mm to (101.4, 112.0), turned to 0 degrees
- moved Q6 2.48 mm to (176.3, 61.7), turned to 180 degrees
- moved Q7 2.48 mm to (106.5, 62.8), turned to 180 degrees
- moved D5 1.91 mm to (173.0, 82.3), turned to 90 degrees
- moved D6 1.91 mm to (179.0, 82.3), turned to 90 degrees
- moved D10 1.90 mm to (115.2, 103.5), turned to 90 degrees
- moved D9 1.90 mm to (109.2, 103.5), turned to 90 degrees
- moved D7 1.85 mm to (165.1, 103.5), turned to 90 degrees
- moved D8 1.85 mm to (171.0, 103.5), turned to 90 degrees
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Connections:
- net /LED1 renamed /LED A
- net /LED2 renamed /LED B
- net /LED3 renamed /LED C
- net /LED4 renamed /LED D
Routing:
- net +5V: track 32.4 -> 271.7 mm
- net Net-(D10-A): track 0.00 -> 138.0 mm
- net Net-(D1-A): track 27.6 -> 155.6 mm
- net Net-(D11-A): track 44.0 -> 133.9 mm, vias 0 -> 2
- net /LED A: track 0.00 -> 88.6 mm
- net Net-(Q8-C): track 0.00 -> 86.7 mm
- net /LED B: track 0.00 -> 45.6 mm
- net Net-(Q1-C): track 0.00 -> 25.0 mm
- net Net-(Q2-C): track 0.00 -> 22.7 mm
- net /DET1: track 19.4 -> 41.8 mm
- net Net-(D7-K): track 0.00 -> 20.4 mm
- net Net-(D1-K): track 0.00 -> 18.7 mm
- net Net-(Q3-C): track 14.5 -> 31.6 mm
- net Net-(Q5-B): track 0.00 -> 16.0 mm
- net Net-(Q8-B): track 0.00 -> 15.0 mm
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Other:
- board text added: "+5V"
- board text added: "1"
- board text added: "2"
- board text added: "A"
- board text added: "A2"
- board text added: "B"
- board text added: "B1"
- board text added: "B2"
- board text added: "C"
- board text added: "C1"
- board text added: "C2"
- board text added: "D"
- board text added: "D1"
- board text added: "D2"
- board text added: "GND"
- board text added: "WalletVac Neck Detector Jan. 2025 Carl Raymond"
