File: Detector/Detector.kicad_sch (KiCad schematic)
At the start: 52 parts, among them J1 Power, J2 Signal, Q1 2N3904, Q2 2N3904, Q3 2N3904, Q4 2N3904, Q5 2N3906, Q6 2N3906, Q7 2N3906, Q8 2N3904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

Commit message: Update detector borad
Parts:
- U1, U2: value TSOP343xx -> TSOP34338
Connections:
- net LED1 renamed LED A
- net LED2 renamed LED B
- net LED3 renamed LED C
- net LED4 renamed LED D
- no-connect marks 0 -> 1
Changed lines of the file:
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@@
 		(color 0 0 0 0)
 	)
+	(no_connect
+		(at 236.22 55.88)
+	)
 	(wire
 		(pts
@@
 		)
 	)
-	(label "LED4"
+	(label "LED D"
 		(at 240.03 66.04 0)
 		(fields_autoplaced yes)
@@
 		)
 	)
-	(label "LED4"
+	(label "LED D"
 		(at 16.51 175.26 0)
 		(fields_autoplaced yes)
@@
 		)
 	)
-	(label "LED3"
+	(label "LED C"
 		(at 16.51 168.91 0)
 		(fields_autoplaced yes)
@@
 		)
 	)
-	(label "LED1"
+	(label "LED A"
 		(at 240.03 58.42 0)
 		(fields_autoplaced yes)
@@
 		)
 	)
-	(label "LED2"
+	(label "LED B"
 		(at 16.51 162.56 0)
 		(fields_autoplaced yes)
@@
 		)
 	)
-	(label "LED3"
+	(label "LED C"
 		(at 240.03 63.5 0)
 		(fields_autoplaced yes)
@@
 		)
 	)
-	(label "LED1"
+	(label "LED A"
 		(at 16.51 156.21 0)
 		(fields_autoplaced yes)
@@
 		)
 	)
-	(label "LED2"
+	(label "LED B"
 		(at 240.03 60.96 0)
 		(fields_autoplaced yes)
@@
 			)
 		)
-		(property "Value" "TSOP343xx"
+		(property "Value" "TSOP34338"
 			(at 157.015 119.38 0)
 			(effects
@@
 			)
 		)
-		(property "Value" "TSOP343xx"
+		(property "Value" "TSOP34338"
 			(at 157.015 90.17 0)
 			(effects
